File: board/ComfortMaps.brd (EAGLE design)
At the start: 96.8 x 49.3 mm, 50 parts, among them J1 PROG_HDR, U1 ADXL362, U2 ATTINY2313, U3 ADP160-3.3, U4 MCP73833, X1 RASPI_GPIO_B+#_PIN

Commit message: v6 board
Parts:
- removed C6: 10uF, SparkFun-Capacitors:0603
- removed D3: RED, SparkFun-LED:LED-0603
- removed D4: GREEN, SparkFun-LED:LED-0603
- removed D5: Yellow, SparkFun-LED:LED-0603
- removed J2: (no value), SparkFun-Connectors:JST-2-SMD
- removed J4: (no value), SparkFun-Connectors:1X02_NO_SILK
- removed R10: THERM, SparkFun-Resistors:AXIAL-0.3
- removed R11: 10k, SparkFun-Resistors:0603
- removed R12: 1k, SparkFun-Resistors:AXIAL-0.3
- removed R4: 10k, SparkFun-Resistors:0603-RES
- removed R5, R6, R7: 1.5k, SparkFun-Resistors:0603
- removed R8: 1k, SparkFun-Resistors:0603
- removed S6: MA12RTR, SparkFun-Switches:SWITCH_SPST_SMD_A
- removed U4: MCP73833, SparkFun-IC-Power:DFN-10
- added C10, C9: 4.7uF, SparkFun-Capacitors:0603
- added C11, C7, C8: 22uF, SparkFun-Capacitors:0805
- added D10, D9: 3A/40V/500mV, SparkFun-DiscreteSemi:SMA-DIODE
- added D11: RED, SparkFun-LED:LED-0603
- added D8: BLUE, SparkFun-LED:LED-0603
- added J5: PTH, SparkFun-Connectors:1X02
- added J6: JST, SparkFun-Connectors:JST-2-SMD
- added L1: 2.2UH3A, SparkFun-Coils:INDUCTOR_4X4MM
- added R20: 1k, SparkFun-Resistors:0603
- added R21, R25: 750K, SparkFun-Resistors:0603
- added R22: 100k, SparkFun-Resistors:0603
- added R24: 4.7k, SparkFun-Resistors:0603
- added RPROG: 2.0k, SparkFun-Resistors:0603
- added S7: MA12RTR, SparkFun-Switches:SWITCH_SPST_SMD_A
- added U5: MCP73831, SparkFun-IC-Power:SOT23-5
- added U6: PAM2401, SparkFun-IC-Power:MSOP8
- moved C5 74.5 mm to (65.8, 37.1)
- moved U$3 21.1 mm to (40.2, 1.09)
Connections:
- removed net N$11: D4.C, R6.1
- removed net N$12: D5.C, R5.1
- removed net N$15: J2.2, S6.1
- removed net PG: R7.2, U4.P$7
- removed net PROG: R12.P$2, R8.2, U4.P$6
- removed net STAT1: R5.2, U4.P$3
- removed net STAT2: R6.2, U4.P$4
- removed net THERM: R10.P$2, R11.2, U4.P$8
- removed net TX0: X1.10
- removed net VDD: C5.1, D3.A, D4.A, D5.A, U4.P$1, U4.P$2, X2.A4B9, X2.B4A9
- removed net V_BATT: C2.1, C6.1, J4.1, Q1.3, R1.1, S6.2, U3.1, U3.3, U4.P$10, U4.P$9
- new net 5V: C7.1, C8.1, D10.C, D11.A, D9.C, R13.2, R14.2, R15.2, R16.2, R21.2, R9.2, U6.7, X1.2, X1.4
- new net 5VIN: C5.1, C9.1, R20.2, U5.4, X2.A4B9, X2.B4A9
- new net EN: R25.1, U6.2
- new net N$10: RPROG.1, U5.5
- new net N$13: D8.C, U5.1
- new net N$17: R21.1, R22.2, U6.5
- new net N$18: L1.P$2, U6.1
- new net N$19: U6.6
- new net N$21: D11.C, R24.2
- new net N$22: D8.A, R20.1
- new net VBATT: C10.1, C11.1, C2.1, L1.P$1, Q1.3, R1.1, R25.2, S7.2, U3.1, U3.3, U5.3, U6.3
- net 3.3V: no longer R13.2, R14.2, R15.2, R16.2, R4.1, R9.2
- net GND: now also C10.2, C11.2, C7.2, C8.2, C9.2, D10.A, D9.A, J5.2, J6.1, R22.1, R24.1, RPROG.2, U5.2, U6.4, U6.8; no longer C6.2, J2.1, J4.2, R10.P$1, R11.1, R12.P$1, R8.1, U4.P$11, U4.P$5
- net N$9: now also J5.1, J6.2, S7.1; no longer D3.C, R7.1
- net RXI: no longer R4.2, X1.8
- net VOUT: no longer X1.2, X1.4
Routing:
- net VBATT: track 0.00 -> 189.8 mm, vias 0 -> 4
- net V_BATT: track 175.5 -> 0.00 mm, vias 2 -> 0
- net 5V: track 0.00 -> 94.3 mm, vias 0 -> 1
- net GND: track 379.8 -> 466.4 mm, vias 5 -> 7
- net 5VIN: track 0.00 -> 59.7 mm, vias 0 -> 3
- net N$9: track 0.00 -> 34.9 mm
- net VDD: track 34.0 -> 0.00 mm
- net N$15: track 27.6 -> 0.00 mm
- net N$13: track 0.00 -> 20.9 mm, vias 0 -> 2
- net N$18: track 0.00 -> 18.2 mm
- net 3.3V: track 93.6 -> 81.4 mm
- net EN: track 0.00 -> 8.68 mm, vias 0 -> 2
- net VOUT: track 64.0 -> 58.7 mm
- net N$17: track 0.00 -> 4.22 mm
- net N$10: track 0.00 -> 3.48 mm
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Other:
- board text added: "Comfort Maps Samuel Clay V6 2020-05-15"
- board text removed: "Comfort Maps Samuel Clay V5 2020-03-02"
